File: KiCAD/BT-E6001/BMS.kicad_sch (KiCad schematic)
At the start: 275 parts, among them CN001 CN001, CN003 S04B-ZESK-2D_T__LF__SN_, CN004 S04B-ZESK-2D_T__LF__SN_, CN2 CN002, IC002 TPS7A1633DGNT / 738 PPNQ or 7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, J1 -, J2 Rx, J3 Tx, J4 +, Q001 Q_PNP, Q002 Q_PNP, Q003 Q_PNP, Q004 Q_PNP, Q005 Q_PNP, Q006 ATP304-TL-H, Q007 ATP304-TL-H, Q008 ATP304-TL-H, Q009 ATP304-TL-H, Q010 ATP304-TL-H, Q011 ATP304-TL-H, Q013 Q_PNP, Q014 Q_NPN, Q015 Q_NPN, Q016 Q_NPN, Q017 Q_NPN, Q018 Q_NPN, Q019 Q_NPN, Q020 Q_NPN, Q021 Q_NPN, Q022 Q_NPN, Q023 Q_NPN, Q024 Q_NPN, Q025 Q_NPN, Q026 Q_PMOS, Q027 Q_PMOS, Q028 Q_PMOS, Q12 Q_PNP, Q29 Q_NMOS, U1 BQ77PL900DL

Commit message: Update KiCAD
Parts:
- added CN5: CN005, Connector_Wire:SolderWire-2.5sqmm_1x01_D2.4mm_OD4.4mm, symbol Connector_Generic:Conn_01x01
- added R102, R103: 1m, symbol Device:R_Small
- added TH003: NTC 10K, SMD0603, symbol Device:Thermistor
- added U2: R2A240, Package_QFP:LQFP-48_7x7mm_P0.5mm, symbol MCU_R2A240:R2A240_60F020
- TH001, TH002: footprint (none) -> THT
Connections:
- net IC003_PIN10 is gone; now on net GND: C51.2, R98.1
- net GND: now also CN5.1 (Pin_1), R102.2, R103.2, TH003.2; no longer J1.1 (Pin_1)
- net IC003_PIN04: now also TH003.1
- new net: J1.1 (Pin_1), R102.1, R103.1
Other:
- note added: "3.6V"
- note added: "36V"
- note added: "BATTERY PACK / CHARGER CONNECTOR"
- note added: "LION-CELL CONNECTOR"
- note added: "next to mosfets Q006..."
- note removed: "BATTERY PACK CONNECTOR"
- moved on the sheet: C1, C10, C11, C12, C13, C14, C15, C16, C17, C18, C2, C25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

Commit message: upd
Parts:
- renumbered U2 to IC003
